Commit message: updated code with gazebo xml files

File: ros2_robot/src/my_robot_description/urdf/common_properties.xacro (robot description, xacro)
@@ -10,3 +10,30 @@
         <color rgba="0.5 0 0 1" />
     </material>
+    <xacro:macro name="box_inertia" params="m l w h xyz rpy" >
+        <inertial>
+            <origin xyz="${xyz}" rpy="${rpy}" />
+            <mass value="${m}"  />
+            <inertia ixx="${(m/12) * (h*h + l*l)}" ixy="0.0" ixz="0.0"
+                     iyy="${(m/12) * (w*w + l*l)}" iyz="0.0"
+                     izz="${(m/12) * (w*w + h*h)}"/>
+        </inertial>
+    </xacro:macro>
+    <xacro:macro name="cylinder_inertia" params="m r h xyz rpy" >
+        <inertial>
+            <origin xyz="${xyz}" rpy="${rpy}" />
+            <mass value="${m}"  />
+            <inertia ixx="${(m/12) * (3*r*r + h*h)}" ixy="0.0" ixz="0.0"
+                     iyy="${(m/12) * (3*r*r + h*h)}" iyz="0.0"
+                     izz="${(m/2) * (r*r)}"/>
+        </inertial>
+    </xacro:macro>
+    <xacro:macro name="sphere_inertia" params="m r xyz rpy" >
+        <inertial>
+            <origin xyz="${xyz}" rpy="${rpy}" />
+            <mass value="${m}"  />
+            <inertia ixx="${2/5 * (m * r * r)}" ixy="0.0" ixz="0.0"
+                     iyy="${2/5 * (m * r * r)}" iyz="0.0"
+                     izz="${2/5 * (m * r * r)}"/>
+        </inertial>
+    </xacro:macro>
 </robot>

File: ros2_robot/src/my_robot_description/urdf/mobile_base.xacro (robot description, xacro)
@@ -6,4 +6,5 @@
     <xacro:property name="wheel_radius" value="0.1" />
     <xacro:property name="wheel_length" value="0.05" />
+    <!-- all parameters were multiplied by 2 to increase the inertia and reduce drift when robot is static -->
     <!--Creating a link-->
     <link name="base_link">
@@ -18,4 +19,13 @@
             <material name="blue" />
         </visual>
+        <collision>
+            <geometry>
+                <box size="${base_length} ${base_width} ${base_height}" />
+            </geometry>
+            <origin xyz="0 0 ${base_height / 2.0}" rpy="0 0 0" />
+        </collision>
+        <xacro:box_inertia m="5.0"
+                           l="${2 * base_length}" w="${2 * base_width}" h="${2 * base_height}"
+                           xyz="0 0 ${base_height / 2.0}" rpy="0 0 0" />
     </link>
     <link name="base_footprint" />
@@ -29,4 +39,12 @@
                 <material name="green" />
             </visual>
+            <collision>
+                <geometry>
+                    <cylinder radius="${wheel_radius}" length="${wheel_length}"/>
+                </geometry>
+                <origin xyz="0 0 0" rpy="${pi /2} 0 0" />
+            </collision>
+            <xacro:cylinder_inertia m="1.0" r="${2 * wheel_radius}" h="${2 * wheel_length}"
+                                    xyz="0 0 0" rpy="${pi /2} 0 0" />
         </link>
     </xacro:macro>
@@ -59,4 +77,12 @@
             <material name="red" />
         </visual>
+        <collision>
+            <geometry>
+                <sphere radius="${wheel_radius / 2.0}" />
+            </geometry>
+            <origin xyz="0 0 0" rpy="0 0 0" />
+        </collision>
+        <xacro:sphere_inertia m="0.5" r="${2 * wheel_radius / 2.0}"
+                              xyz="0 0 0" rpy="0 0 0" />
     </link>
     <joint name="base_joint" type="fixed">

File: ros2_robot/src/my_robot_description/urdf/my_robot.urdf.xacro (robot description, xacro)
@@ -5,3 +5,4 @@
     <xacro:include filename="common_properties.xacro" />
     <xacro:include filename="mobile_base.xacro" />
+    <xacro:include filename="test_parrot_gazebo.xacro" />
 </robot>
